File: PCBV2/MCU&Power.sch (KiCad schematic (older format))
At the start: 30 parts, among them J1 USB_B_Micro, J2 Conn_01x02_Female, Q43 PSMN5R2-60YL, T1 750312367, U5 LT3759, U7 TPS2514

Commit message: Clean up for readability
Other:
- note added: "HV Generator"
- note added: "MCU"
- note added: "USB"
- moved on the sheet: A1, C11, C12, C13, C14, C15, C17, C18, C19, C20, C21, C9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
