File: PCBV2/PCBV2.sch (KiCad schematic (older format))
At the start: 106 parts, among them Q1 Q_NPN_BEC, Q10 Q_NPN_BEC, Q11 Q_NPN_BEC, Q12 Q_NPN_BEC, Q13 Q_NPN_BEC, Q14 Q_NPN_BEC, Q15 Q_NPN_BEC, Q16 Q_NPN_BEC, Q17 Q_NPN_BEC, Q18 Q_NPN_BEC, Q19 Q_NPN_BEC, Q2 Q_NPN_BEC, Q20 Q_NPN_BEC, Q21 Q_NPN_BEC, Q22 Q_NPN_BEC, Q23 Q_NPN_BEC, Q24 Q_NPN_BEC, Q25 Q_NPN_BEC, Q26 Q_NPN_BEC, Q27 Q_NPN_BEC, Q28 Q_NPN_BEC, Q29 Q_NPN_BEC, Q3 Q_NPN_BEC, Q30 Q_NPN_BEC, Q31 Q_NPN_BEC, Q32 Q_NPN_BEC, Q33 Q_NPN_BEC, Q34 Q_NPN_BEC, Q35 Q_NPN_BEC, Q36 Q_NPN_BEC, Q37 Q_NPN_BEC, Q38 Q_NPN_BEC, Q39 Q_NPN_BEC, Q4 Q_NPN_BEC, Q40 Q_NPN_BEC, Q5 Q_NPN_BEC, Q6 Q_NPN_BEC, Q7 Q_NPN_BEC, Q8 Q_NPN_BEC, Q9 Q_NPN_BEC, U1 PCA9685BS, U2 PCA9685BS, U3 PCA9685BS

Commit message: Clean up for readability
Parts:
- removed C? (x4): 0.1uF, Capacitor_SMD:C_0603_1608Metric, symbol Device:C_Small
- removed D? (x4): IN-PI55QATPRPGPBPW, LED_SMD:LED_Inolux_IN-PI554FCH_PLCC4_5.0x5.0mm_P3.2mm, symbol PCBV2-rescue:IN-PI55QATPRPGPBPW-LED
Other:
- note added: "DRIVERS"
- note added: "MOSFETS"
- note added: "Nixie Tubes"
- note added: "RGB LED"
- moved on the sheet: C1, C2, C3, C4, D1, D2, D3, D4
